Commit message: “路径规划算法优化”

File: src/arm_description/urdf/blueberry_arm.urdf.xacro (robot description, xacro)
@@ -69,5 +69,5 @@
     <origin xyz="0 0 0.083" rpy="0 0 0"/>  <!-- 位于基座顶部中心 -->
     <axis xyz="0 0 1"/>  <!-- 绕Z轴旋转 -->
-    <limit lower="-3.14" upper="3.14" effort="100" velocity="1.0"/>  <!-- 360°旋转 -->
+    <limit lower="-2.0944" upper="2.0944" effort="100" velocity="1.0"/>  <!-- 360°旋转 -->
   </joint>
   <!-- 关节1 (俯仰) -->
@@ -96,5 +96,5 @@
     <origin xyz="0 0 0.02" rpy="0 -1.57 0"/>  <!-- 位于旋转圆盘顶部 -->
     <axis xyz="0 1 0"/>  <!-- 绕Y轴俯仰 -->
-    <limit lower="0" upper="1.57" effort="50" velocity="0.5"/>  <!-- -90°~90° -->
+    <limit lower="-2.0944" upper="2.0944" effort="50" velocity="0.5"/>  <!-- -90°~90° -->
   </joint>
   <!-- 关节2 (俯仰) -->
@@ -123,5 +123,5 @@
     <origin xyz="0.129 0 0" rpy="0 0 0"/>  <!-- 连接arm1末端 -->
     <axis xyz="0 1 0"/>  <!-- 绕Y轴俯仰 -->
-    <limit lower="0" upper="1.57" effort="50" velocity="0.5"/>
+    <limit lower="-2.0944" upper="2.0944" effort="50" velocity="0.5"/>
   </joint>
   <!-- 关节3 (俯仰) -->
@@ -150,5 +150,5 @@
     <origin xyz="0.129 0 0" rpy="0 0 0"/>  <!-- 连接arm2末端 -->
     <axis xyz="0 1 0"/>  <!-- 绕Y轴俯仰 -->
-    <limit lower="0" upper="1.57" effort="30" velocity="0.5"/>
+    <limit lower="-2.0944" upper="2.0944" effort="30" velocity="0.5"/>
   </joint>
   <!-- 末端执行器 -->

Commit message: “”

File: src/arm_description/urdf/blueberry_arm.urdf.xacro (robot description, xacro)
@@ -129,14 +129,14 @@
     <visual>
       <geometry>
-        <box size="0.071 0.04 0.04"/>  <!-- 长171mm (含夹爪) -->
-      </geometry>
-      <origin xyz="0.0355 0 0" rpy="0 0 0"/>
+        <box size="0.0525 0.04 0.04"/>  <!-- 长171mm (含夹爪) -->
+      </geometry>
+      <origin xyz="0.02625 0 0" rpy="0 0 0"/>
       <material name="silver"/>
     </visual>
     <collision>
       <geometry>
-        <box size="0.071 0.04 0.04"/>
-      </geometry>
-      <origin xyz="0.0355 0 0" rpy="0 0 0"/>
+        <box size="0.0525 0.04 0.04"/>
+      </geometry>
+      <origin xyz="0.02625 0 0" rpy="0 0 0"/>
     </collision>
     <inertial>
@@ -156,14 +156,14 @@
     <visual>
       <geometry>
-        <cylinder length="0.10" radius="0.02"/>  <!-- 简化表示 -->
-      </geometry>
-      <origin xyz="0.05 0 0" rpy="0 1.57 0"/>
+        <cylinder length="0.06" radius="0.0125"/>  <!-- 简化表示 -->
+      </geometry>
+      <origin xyz="0.03 0 0" rpy="0 1.57 0"/>
       <material name="blue"/>
     </visual>
     <collision>
       <geometry>
-        <cylinder length="0.10" radius="0.02"/>
-      </geometry>
-      <origin xyz="0.05 0 0" rpy="0 1.57 0"/>
+        <cylinder length="0.06" radius="0.0125"/>
+      </geometry>
+      <origin xyz="0.03 0 0" rpy="0 1.57 0"/>
     </collision>
     <inertial>
@@ -175,5 +175,5 @@
     <parent link="arm3_link"/>
     <child link="end_effector"/>
-    <origin xyz="0.071 0 0" rpy="0 0 0"/>  <!-- 位于arm3末端 -->
+    <origin xyz="0.0525 0.04 -0.0275" rpy="0 0 0"/>  <!-- 位于arm3末端 -->
   </joint>
   <!-- 相机 -->
@@ -181,5 +181,5 @@
     <visual>
       <geometry>
-        <box size="0.0155 0.0653 0.0225"/>
+        <box size="0.0155 0.0653 0.031"/>
       </geometry>
       <origin xyz="0 0 0" rpy="0 0 0"/>
@@ -188,5 +188,5 @@
     <collision>
       <geometry>
-        <box size="0.0155 0.0653 0.0225"/>
+        <box size="0.0155 0.0653 0.031"/>
       </geometry>
       <origin xyz="0 0 0" rpy="0 0 0"/>
@@ -200,5 +200,5 @@
     <parent link="arm3_link"/>
     <child link="camera_link"/>
-    <origin xyz="0.071 0 0.03125" rpy="0 0 0"/>
+    <origin xyz="0.0525 0 0.048" rpy="0 0 0"/>
   </joint>
   <!-- 光学坐标系定义 -->
